File: smart_toilet/smart_toilet.kicad_sch (KiCad schematic)
At the start: 54 parts, among them J1 Conn_01x02, J2 Conn_01x04, J3 Conn_01x04, J3 USB_C_Receptacle_USB2.0, Q1 BC860, Q1 MMBT5550L, Q2 BC860, Q2 MMBT5550L, SW2 SW_Omron_B3FS, U1 ESP32-WROOM-32D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

Commit message: UPDATED PCB
Parts:
- added H1, H2, H3, H4: MountingHole, MountingHole:MountingHole_3.5mm, symbol Mechanical:MountingHole
Connections:
- net S+: now also J3.3 (Pin_3); no longer J3.2 (Pin_2)
- net S+_1: no longer J2.2 (Pin_2)
- net S-: now also J3.2 (Pin_2); no longer J3.3 (Pin_3)
- net S-_1: now also J2.2 (Pin_2)
- net SCK1: now reaches U1.11 (IO26)
- net SCK1: now also U1.11 (PD_SCK)
- net DOUT1: now reaches U1.12 (IO27)
- net DOUT1: now also U1.12 (DOUT)
- net DOUT2: now reaches U1.27 (IO16)
- net DOUT2: now also U2.12 (DOUT)
- net SCK2: now reaches U1.28 (IO17)
- net SCK2: now also U2.11 (PD_SCK)
- no-connect marks 27 -> 31
Other:
- note added: "HX711"
- note added: "PROGRAMMING"
- note added: "USB-C"
- moved on the sheet: C1, C10, C11, C12, C17, C18, C19, C2, C3, C4, D2, D4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
