File: smart_toilet/smart_toilet.kicad_sch (KiCad schematic)
At the start: 59 parts, among them J1 Conn_01x02, J2 Conn_01x04, J3 Conn_01x04, J3 USB_C_Receptacle_USB2.0, Q1 BC860, Q1 MMBT5550L, Q2 BC860, Q2 MMBT5550L, SW2 SW_Omron_B3FS, U1 ESP32-WROOM-32D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

Commit message: updated
Parts:
- added C6, C8: 10uF, Capacitor_SMD:C_0603_1608Metric_Pad1.08x0.95mm_HandSolder, symbol Device:C_Small
- added R5: 1.6K, Resistor_SMD:R_0805_2012Metric_Pad1.20x1.40mm_HandSolder, symbol Device:R
- added TP1, TP10, TP11, TP12, TP13, TP14, TP15, TP16, TP17, TP18, TP19, TP2, TP20, TP21, TP3, TP4, TP5, TP6, TP7, TP8, TP9: TestPoint, TestPoint:TestPoint_Pad_D1.0mm, symbol Connector:TestPoint
- added U3: TP4057, Package_TO_SOT_SMD:SOT-23-6_Handsoldering, symbol TP4057:TP4057
- C1, C10, C3, C4: value C_Small -> 10uF
- C11, C2, C5, C6: value C_Small -> 0.1uF
- R1, R3: value 1K -> 20K; footprint Resistor_SMD:R_0603_1608Metric_Pad0.98x0.95mm_HandSolder -> Resistor_SMD:R_0805_2012Metric_Pad1.20x1.40mm_HandSolder
- R10, R11, R5, R6: value R_US -> 1.2K
- R19, R7: footprint Resistor_SMD:R_0603_1608Metric_Pad0.98x0.95mm_HandSolder -> Resistor_SMD:R_0805_2012Metric_Pad1.20x1.40mm_HandSolder
- R2, R4: value 1K -> 8.2K; footprint Resistor_SMD:R_0603_1608Metric_Pad0.98x0.95mm_HandSolder -> Resistor_SMD:R_0805_2012Metric_Pad1.20x1.40mm_HandSolder
Connections:
- net +BATT: now also C8.2, U3.3 (BAT)
- net GND: now also R2.1, R4.1, U1.5 (AGND), U2.5 (AGND), C6.1, C8.1, R5.1, U3.2 (GND)
- net VBUS: now also C6.2, U3.4 (VCC)
- net at U1.10 (IO25): now also TP12.1
- net at U1.13 (IO14): now also TP5.1
- net at U1.14 (IO12): now also TP3.1
- net at U1.16 (IO13): now also TP4.1
- net at U1.17 (SHD/SD2): now also TP18.1
- net at U1.18 (SWP/SD3): now also TP19.1
- net at U1.19 (SCS/CMD): now also TP21.1
- net at U1.20 (SCK/CLK): now also TP20.1
- net at U1.21 (SDO/SD0): now also TP16.1
- net at U1.22 (SDI/SD1): now also TP17.1
- net at U1.23 (IO15): now also TP6.1
- net at U1.26 (IO4): now also TP1.1
- net at U1.29 (IO5): now also TP2.1
- net at U1.30 (IO18): now also TP7.1
- net at U1.31 (IO19): now also TP8.1
- net at U1.33 (IO21): now also TP9.1
- net at U1.36 (IO22): now also TP10.1
- net at U1.37 (IO23): now also TP11.1
- net at U1.7 (IO35): now also TP15.1
- net at U1.8 (IO32): now also TP13.1
- net at U1.9 (IO33): now also TP14.1
- new net: R5.2, U3.6 (PROG)
- no-connect marks 31 -> 13
Other:
- moved on the sheet: C2, C5, R5, R6
