File: smart_toilet/_autosave-smart_toilet.kicad_sch (KiCad schematic)
At the start: 59 parts, among them J1 Conn_01x02, J2 Conn_01x04, J3 Conn_01x04, J3 USB_C_Receptacle_USB2.0, Q1 BC860, Q1 MMBT5550L, Q2 BC860, Q2 MMBT5550L, SW2 SW_Omron_B3FS, U1 ESP32-WROOM-32D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

Commit message: UPDATED
Parts:
- added C6, C8: 10uF, Capacitor_SMD:C_0603_1608Metric_Pad1.08x0.95mm_HandSolder, symbol Device:C_Small
- added R5: 1.6K, Resistor_SMD:R_0603_1608Metric_Pad0.98x0.95mm_HandSolder, symbol Device:R
- added U3: TP4057, Package_TO_SOT_SMD:SOT-23-6_Handsoldering, symbol TP4057:TP4057
Connections:
- net +BATT: now also C8.2, U3.3 (BAT)
- net GND: now also C6.1, C8.1, R5.1, U3.2 (GND)
- net VBUS: now also C6.2, U3.4 (VCC)
- new net: R5.2, U3.6 (PROG)
- no-connect marks 31 -> 33
