File: smart_toilet/smart_toilet.kicad_pcb (KiCad board)
At the start: 2 copper layers, 90.1 x 56 mm, 54 parts, among them J1 Conn_01x02, J2 Conn_01x04, J3 Conn_01x04, J5 USB_C_Receptacle_USB2.0, Q1 BC860, Q2 BC860, Q3 MMBT5550L, Q4 MMBT5550L, SW1 SW_Omron_B3FS, U1 HX711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

Commit message: UPDATED PCB
Parts:
- added H1: MountingHole, MountingHole:MountingHole_3.5mm, F.Cu at (112.7, 83.2)
- added H2: MountingHole, MountingHole:MountingHole_3.5mm, F.Cu at (175.4, 83.0)
- added H3: MountingHole, MountingHole:MountingHole_3.5mm, F.Cu at (114.3, 122.0)
- added H4: MountingHole, MountingHole:MountingHole_3.5mm, F.Cu at (175.8, 122.5)
- moved R14 20.3 mm to (153.5, 105.0), turned to 90 degrees
- moved R15 18.0 mm to (116.5, 109.1), turned to 180 degrees
- moved R16 15.3 mm to (116.5, 107.1), turned to 0 degrees
- moved D2 14.3 mm to (151.5, 105.0), turned to 90 degrees
- moved SW1 13.4 mm to (130.5, 97.0)
- moved C9 12.9 mm to (131.5, 92.2)
- moved Q3 11.0 mm to (140.7, 106.1), turned to 90 degrees
- moved C3 10.7 mm to (170.3, 104.2)
- moved C4 10.7 mm to (170.3, 100.4)
- moved C6 10.7 mm to (165.8, 96.4)
- moved Q1 10.7 mm to (167.1, 104.2)
- moved R3 10.7 mm to (168.1, 100.4)
- moved R4 10.7 mm to (165.9, 100.4)
- moved R5 10.7 mm to (169.1, 97.2)
- moved R6 10.7 mm to (169.1, 95.4)
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Connections:
- J2 pad 2: S+_1 -> S-_1
- J3 pad 2: S+ -> S-
- J3 pad 3: S- -> S+
- U1 pad 11: unconnected-(U1-PD_SCK-Pad11) -> SCK1
- U1 pad 12: unconnected-(U1-DOUT-Pad12) -> DOUT1
- U2 pad 11: unconnected-(U2-PD_SCK-Pad11) -> SCK2
- U2 pad 12: unconnected-(U2-DOUT-Pad12) -> DOUT2
- U4 pad 11: unconnected-(U4-IO26-Pad11) -> SCK1
- U4 pad 12: unconnected-(U4-IO27-Pad12) -> DOUT1
- U4 pad 27: unconnected-(U4-IO16-Pad27) -> DOUT2
- U4 pad 28: unconnected-(U4-IO17-Pad28) -> SCK2
Routing:
- net +5V: track 13.7 -> 130.4 mm, vias 0 -> 2
- net +3.3V: track 0.00 -> 56.1 mm
- net TX0: track 0.00 -> 48.9 mm, vias 0 -> 2
- net DTR: track 4.34 -> 49.2 mm, vias 0 -> 2
- net RX0: track 0.00 -> 42.8 mm, vias 0 -> 2
- net RTS: track 2.16 -> 40.5 mm, vias 0 -> 2
- net BTSENS: track 1.75 -> 39.0 mm, vias 0 -> 2
- net ESP_EN: track 0.00 -> 33.1 mm
- net DOUT1: track 0.00 -> 29.4 mm, vias 0 -> 2
- net SCK1: track 0.00 -> 29.3 mm, vias 0 -> 2
- net DN: track 0.00 -> 25.3 mm, vias 0 -> 2
- net DP: track 0.00 -> 24.0 mm, vias 0 -> 2
- net DOUT2: track 0.00 -> 19.4 mm, vias 0 -> 2
- net SCK2: track 0.00 -> 18.8 mm, vias 0 -> 2
- net S+: track 0.00 -> 18.7 mm, vias 0 -> 1
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- added copper zone on F.Cu, net +5V
- added copper zone on F.Cu, net +BATT
- added copper zone on F.Cu, net /SW
- added copper zone on B.Cu, net GND
- added copper zone on F.Cu, net GND
- added copper zone on F.Cu, net Net-(JP2-B)

Commit message: UPDATED
Parts:
- added C17: 10uF, Capacitor_SMD:C_0603_1608Metric_Pad1.08x0.95mm_HandSolder, F.Cu at (124.4, 102.0)
- added C18: 10uF, Capacitor_SMD:C_0603_1608Metric_Pad1.08x0.95mm_HandSolder, F.Cu at (124.4, 109.0)
- added R19: 1.6K, Resistor_SMD:R_0603_1608Metric_Pad0.98x0.95mm_HandSolder, F.Cu at (121.6, 105.5)
- added U7: TP4057, Package_TO_SOT_SMD:SOT-23-6_Handsoldering, F.Cu at (124.4, 105.5)
- moved R17 1.81 mm to (114.8, 105.2)
- moved R18 1.81 mm to (114.8, 103.2)
- moved R15 1.81 mm to (114.8, 109.2)
- moved R16 1.81 mm to (114.8, 107.2)
Routing:
- net VBUS: track 0.00 -> 25.3 mm, vias 0 -> 2
- net unconnected-(J5-SHIELD-PadS1): track 0.00 -> 17.0 mm
- net VCC: track 8.24 -> 24.2 mm
- net BTSENS: track 39.0 -> 44.1 mm
- net TX0: track 48.9 -> 46.6 mm
- net Net-(U7-PROG): track 0.00 -> 2.03 mm
- net Net-(J5-CC1): track 5.80 -> 4.06 mm
- net Net-(J5-CC2): track 5.48 -> 3.80 mm
- net RX0: track 42.8 -> 43.4 mm

Commit message: updated
Parts:
- added TP1: TestPoint, TestPoint:TestPoint_Pad_D1.0mm, F.Cu at (154.0, 99.2)
- added TP10: TestPoint, TestPoint:TestPoint_Pad_D1.0mm, F.Cu at (154.0, 86.4)
- added TP11: TestPoint, TestPoint:TestPoint_Pad_D1.0mm, F.Cu at (155.5, 84.9)
- added TP12: TestPoint, TestPoint:TestPoint_Pad_D1.0mm, F.Cu at (131.0, 106.2)
- added TP13: TestPoint, TestPoint:TestPoint_Pad_D1.0mm, F.Cu at (130.8, 103.7)
- added TP14: TestPoint, TestPoint:TestPoint_Pad_D1.0mm, F.Cu at (128.5, 106.2)
- added TP15: TestPoint, TestPoint:TestPoint_Pad_D1.0mm, F.Cu at (128.5, 103.7)
- added TP16: TestPoint, TestPoint:TestPoint_Pad_D1.0mm, F.Cu at (144.8, 104.2)
- added TP17: TestPoint, TestPoint:TestPoint_Pad_D1.0mm, F.Cu at (146.3, 106.4)
- added TP18: TestPoint, TestPoint:TestPoint_Pad_D1.0mm, F.Cu at (139.8, 104.2)
- added TP19: TestPoint, TestPoint:TestPoint_Pad_D1.0mm, F.Cu at (141.0, 106.4)
- added TP2: TestPoint, TestPoint:TestPoint_Pad_D1.0mm, F.Cu at (154.0, 95.4)
- added TP20: TestPoint, TestPoint:TestPoint_Pad_D1.0mm, F.Cu at (143.5, 106.4)
- added TP21: TestPoint, TestPoint:TestPoint_Pad_D1.0mm, F.Cu at (142.3, 104.2)
- added TP3: TestPoint, TestPoint:TestPoint_Pad_D1.0mm, F.Cu at (130.8, 101.4)
- added TP4: TestPoint, TestPoint:TestPoint_Pad_D1.0mm, F.Cu at (138.5, 106.4)
- added TP5: TestPoint, TestPoint:TestPoint_Pad_D1.0mm, F.Cu at (128.5, 101.4)
- added TP6: TestPoint, TestPoint:TestPoint_Pad_D1.0mm, F.Cu at (147.5, 103.9)
- added TP7: TestPoint, TestPoint:TestPoint_Pad_D1.0mm, F.Cu at (156.0, 94.2)
- added TP8: TestPoint, TestPoint:TestPoint_Pad_D1.0mm, F.Cu at (154.0, 92.9)
- added TP9: TestPoint, TestPoint:TestPoint_Pad_D1.0mm, F.Cu at (154.0, 90.4)
- C1, C10, C3, C4: value C_Small -> 10uF
- C11, C2, C5, C6: value C_Small -> 0.1uF
- R1, R3: value 1K -> 20K; footprint Resistor_SMD:R_0603_1608Metric_Pad0.98x0.95mm_HandSolder -> Resistor_SMD:R_0805_2012Metric_Pad1.20x1.40mm_HandSolder
- R10, R11, R5, R6: value R_US -> 1.2K
- R16, R19, R8: footprint Resistor_SMD:R_0603_1608Metric_Pad0.98x0.95mm_HandSolder -> Resistor_SMD:R_0805_2012Metric_Pad1.20x1.40mm_HandSolder
- R2, R4: value 1K -> 8.2K; footprint Resistor_SMD:R_0603_1608Metric_Pad0.98x0.95mm_HandSolder -> Resistor_SMD:R_0805_2012Metric_Pad1.20x1.40mm_HandSolder
- moved Q3 12.6 mm to (151.1, 113.2), turned to -90 degrees
- moved R9 9.73 mm to (147.6, 114.2), turned to 180 degrees
- moved Q4 7.89 mm to (144.1, 113.2), turned to -90 degrees
- moved R12 6.17 mm to (147.6, 112.2), turned to 0 degrees
- moved J3 2.11 mm to (183.8, 104.2)
- moved J2 2.11 mm to (183.8, 116.8)
- moved J5 2.01 mm to (104.2, 103.4)
- moved J1 1.71 mm to (107.2, 113.1)
- moved R19 0.35 mm to (121.2, 105.5)
- moved R16 0.25 mm to (114.8, 107.0)
- moved R8 0.25 mm to (132.8, 113.8)
- moved R7 0.15 mm to (134.8, 113.8)
- moved Q2 0.07 mm to (166.8, 117.2)
Connections:
- R2 pad 1: Net-(U2-AGND) -> GND
- R4 pad 1: Net-(U1-AGND) -> GND
- U1 pad 5: Net-(U1-AGND) -> GND
- U2 pad 5: Net-(U2-AGND) -> GND
- U4 pad 10: unconnected-(U4-IO25-Pad10) -> Net-(U4-IO25)
- U4 pad 13: unconnected-(U4-IO14-Pad13) -> Net-(U4-IO14)
- U4 pad 14: unconnected-(U4-IO12-Pad14) -> Net-(U4-IO12)
- U4 pad 16: unconnected-(U4-IO13-Pad16) -> Net-(U4-IO13)
- U4 pad 17: unconnected-(U4-SHD/SD2-Pad17) -> Net-(U4-SHD/SD2)
- U4 pad 18: unconnected-(U4-SWP/SD3-Pad18) -> Net-(U4-SWP/SD3)
- U4 pad 19: unconnected-(U4-SCS/CMD-Pad19) -> Net-(U4-SCS/CMD)
- U4 pad 20: unconnected-(U4-SCK/CLK-Pad20) -> Net-(U4-SCK/CLK)
- U4 pad 21: unconnected-(U4-SDO/SD0-Pad21) -> Net-(U4-SDO/SD0)
- U4 pad 22: unconnected-(U4-SDI/SD1-Pad22) -> Net-(U4-SDI/SD1)
- U4 pad 23: unconnected-(U4-IO15-Pad23) -> Net-(U4-IO15)
- U4 pad 26: unconnected-(U4-IO4-Pad26) -> Net-(U4-IO4)
- U4 pad 29: unconnected-(U4-IO5-Pad29) -> Net-(U4-IO5)
- U4 pad 30: unconnected-(U4-IO18-Pad30) -> Net-(U4-IO18)
- U4 pad 31: unconnected-(U4-IO19-Pad31) -> Net-(U4-IO19)
- U4 pad 33: unconnected-(U4-IO21-Pad33) -> Net-(U4-IO21)
- U4 pad 36: unconnected-(U4-IO22-Pad36) -> Net-(U4-IO22)
- U4 pad 37: unconnected-(U4-IO23-Pad37) -> Net-(U4-IO23)
- U4 pad 7: unconnected-(U4-IO35-Pad7) -> Net-(U4-IO35)
- U4 pad 8: unconnected-(U4-IO32-Pad8) -> Net-(U4-IO32)
- U4 pad 9: unconnected-(U4-IO33-Pad9) -> Net-(U4-IO33)
Routing:
- net Net-(U4-IO25): track 0.00 -> 24.8 mm, vias 0 -> 2
- net Net-(U4-IO33): track 0.00 -> 24.5 mm, vias 0 -> 2
- net Net-(U4-IO14): track 0.00 -> 22.6 mm, vias 0 -> 2
- net Net-(U4-IO35): track 0.00 -> 22.3 mm, vias 0 -> 2
- net ESP_EN: track 33.1 -> 54.7 mm
- net Net-(U4-IO32): track 0.00 -> 21.4 mm, vias 0 -> 2
- net IO0: track 9.87 -> 24.8 mm
- net +5V: track 130.4 -> 139.2 mm
- net RTS: track 40.5 -> 49.1 mm
- net Net-(U4-IO12): track 0.00 -> 6.57 mm, vias 0 -> 2
- net Net-(U4-SCK/CLK): track 0.00 -> 4.97 mm
- net Net-(U4-SDI/SD1): track 0.00 -> 4.96 mm
- net Net-(U4-SWP/SD3): track 0.00 -> 4.95 mm
- net Net-(U4-IO13): track 0.00 -> 4.93 mm
- net GND: track 9.84 -> 14.7 mm, vias 255 -> 311
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